Commit message: feat: Introduce the Alive pipeline, Synapse interoperability layer, and unified multi-domain RGD structure
This commit represents a foundational step in the evolution of the OpenRGD ecosystem.

• Added the `alive` command: a full cognitive instantiation pipeline that merges
  imported robot descriptions (URDF/USD) with a complete multi-domain RGD seed,
  generating a fully functional RGD profile (00_core → 06_ether).

• Introduced the `synapse` subsystem: a universal interoperability layer designed
  to export OpenRGD into external frameworks (ROS2, Isaac, USD pipelines, etc.).
  Synapse formalizes the concept of “cognitive bridges” that link RGD semantics
  with real-world runtime ecosystems.

• Restructured project layout for clarity, extensibility, and cross-domain alignment:
  - normalized directory structure
  - standardized seed loading paths
  - improved importer pipeline
  - consolidated command registration
  - prepared for future multi-LLM domain agents

• Implemented automatic dependency synchronization:
  - added `tools/generate_requirements.py`
  - workflow now regenerates requirements.txt from pyproject.toml
  - ensures consistent dependency resolution across all environments

Collectively, these changes reinforce OpenRGD’s mission to provide a universal,
interoperable, and future-proof cognitive BIOS for robotics.

And I officially ran out of coffee. At this point I’d happily ask an OpenRGD-powered robot to restock the lab.

File: export/rgd_hardware.xacro (robot description, xacro)
@@ -5,4 +5,52 @@
       <plugin>odrive_can_controller/ODriveCANInterface</plugin>
     </hardware>
+    <joint name="leg_left_hip_yaw">
+      <param name="can_id">0</param>
+      <param name="bus">can0</param>
+      <command_interface name="position"/>
+      <state_interface name="position"/>
+      <state_interface name="velocity"/>
+      <state_interface name="effort"/>
+    </joint>
+    <joint name="leg_left_ankle_pitch">
+      <param name="can_id">0</param>
+      <param name="bus">can0</param>
+      <command_interface name="position"/>
+      <state_interface name="position"/>
+      <state_interface name="velocity"/>
+      <state_interface name="effort"/>
+    </joint>
+    <joint name="leg_right_hip_pitch">
+      <param name="can_id">0</param>
+      <param name="bus">can0</param>
+      <command_interface name="position"/>
+      <state_interface name="position"/>
+      <state_interface name="velocity"/>
+      <state_interface name="effort"/>
+    </joint>
+    <joint name="arm_right_shoulder_roll">
+      <param name="can_id">0</param>
+      <param name="bus">can0</param>
+      <command_interface name="position"/>
+      <state_interface name="position"/>
+      <state_interface name="velocity"/>
+      <state_interface name="effort"/>
+    </joint>
+    <joint name="arm_left_elbow_pitch">
+      <param name="can_id">0</param>
+      <param name="bus">can0</param>
+      <command_interface name="position"/>
+      <state_interface name="position"/>
+      <state_interface name="velocity"/>
+      <state_interface name="effort"/>
+    </joint>
+    <joint name="arm_right_shoulder_pitch">
+      <param name="can_id">0</param>
+      <param name="bus">can0</param>
+      <command_interface name="position"/>
+      <state_interface name="position"/>
+      <state_interface name="velocity"/>
+      <state_interface name="effort"/>
+    </joint>
     <joint name="knee_joint_right">
       <param name="can_id">12</param>
@@ -13,5 +61,53 @@
       <state_interface name="effort"/>
     </joint>
+    <joint name="leg_right_hip_roll">
+      <param name="can_id">0</param>
+      <param name="bus">can0</param>
+      <command_interface name="position"/>
+      <state_interface name="position"/>
+      <state_interface name="velocity"/>
+      <state_interface name="effort"/>
+    </joint>
+    <joint name="leg_left_hip_roll">
+      <param name="can_id">0</param>
+      <param name="bus">can0</param>
+      <command_interface name="position"/>
+      <state_interface name="position"/>
+      <state_interface name="velocity"/>
+      <state_interface name="effort"/>
+    </joint>
+    <joint name="leg_right_knee_pitch">
+      <param name="can_id">0</param>
+      <param name="bus">can0</param>
+      <command_interface name="position"/>
+      <state_interface name="position"/>
+      <state_interface name="velocity"/>
+      <state_interface name="effort"/>
+    </joint>
     <joint name="hip_pitch_right">
+      <param name="can_id">0</param>
+      <param name="bus">can0</param>
+      <command_interface name="position"/>
+      <state_interface name="position"/>
+      <state_interface name="velocity"/>
+      <state_interface name="effort"/>
+    </joint>
+    <joint name="leg_right_ankle_pitch">
+      <param name="can_id">0</param>
+      <param name="bus">can0</param>
+      <command_interface name="position"/>
+      <state_interface name="position"/>
+      <state_interface name="velocity"/>
+      <state_interface name="effort"/>
+    </joint>
+    <joint name="leg_left_knee_pitch">
+      <param name="can_id">0</param>
+      <param name="bus">can0</param>
+      <command_interface name="position"/>
+      <state_interface name="position"/>
+      <state_interface name="velocity"/>
+      <state_interface name="effort"/>
+    </joint>
+    <joint name="leg_left_hip_pitch">
       <param name="can_id">0</param>
       <param name="bus">can0</param>
@@ -29,4 +125,36 @@
       <state_interface name="effort"/>
     </joint>
+    <joint name="arm_left_shoulder_pitch">
+      <param name="can_id">0</param>
+      <param name="bus">can0</param>
+      <command_interface name="position"/>
+      <state_interface name="position"/>
+      <state_interface name="velocity"/>
+      <state_interface name="effort"/>
+    </joint>
+    <joint name="leg_right_hip_yaw">
+      <param name="can_id">0</param>
+      <param name="bus">can0</param>
+      <command_interface name="position"/>
+      <state_interface name="position"/>
+      <state_interface name="velocity"/>
+      <state_interface name="effort"/>
+    </joint>
+    <joint name="arm_left_shoulder_roll">
+      <param name="can_id">0</param>
+      <param name="bus">can0</param>
+      <command_interface name="position"/>
+      <state_interface name="position"/>
+      <state_interface name="velocity"/>
+      <state_interface name="effort"/>
+    </joint>
+    <joint name="arm_right_elbow_pitch">
+      <param name="can_id">0</param>
+      <param name="bus">can0</param>
+      <command_interface name="position"/>
+      <state_interface name="position"/>
+      <state_interface name="velocity"/>
+      <state_interface name="effort"/>
+    </joint>
   </ros2_control>
 </robot>

File: export/rgd_limits.xacro (robot description, xacro)
@@ -1,5 +1,41 @@
 <?xml version="1.0"?>
 <robot xmlns:xacro="http://www.ros.org/wiki/xacro">
-  <xacro:property name="knee_joint_right_effort" value="40.0" />
+  <xacro:property name="leg_left_hip_yaw_effort" value="40.0" />
+  <xacro:property name="leg_left_hip_yaw_velocity" value="0.0" />
+  <xacro:property name="leg_left_hip_yaw_lower" value="-3.14" />
+  <xacro:property name="leg_left_hip_yaw_upper" value="3.14" />
+  <xacro:property name="leg_left_hip_yaw_damping" value="0.0" />
+  <xacro:property name="leg_left_hip_yaw_friction" value="0.0" />
+  <xacro:property name="leg_left_ankle_pitch_effort" value="30.0" />
+  <xacro:property name="leg_left_ankle_pitch_velocity" value="0.0" />
+  <xacro:property name="leg_left_ankle_pitch_lower" value="-3.14" />
+  <xacro:property name="leg_left_ankle_pitch_upper" value="3.14" />
+  <xacro:property name="leg_left_ankle_pitch_damping" value="0.0" />
+  <xacro:property name="leg_left_ankle_pitch_friction" value="0.0" />
+  <xacro:property name="leg_right_hip_pitch_effort" value="80.0" />
+  <xacro:property name="leg_right_hip_pitch_velocity" value="8.0" />
+  <xacro:property name="leg_right_hip_pitch_lower" value="-3.14" />
+  <xacro:property name="leg_right_hip_pitch_upper" value="3.14" />
+  <xacro:property name="leg_right_hip_pitch_damping" value="0.0" />
+  <xacro:property name="leg_right_hip_pitch_friction" value="0.0" />
+  <xacro:property name="arm_right_shoulder_roll_effort" value="18.0" />
+  <xacro:property name="arm_right_shoulder_roll_velocity" value="0.0" />
+  <xacro:property name="arm_right_shoulder_roll_lower" value="-3.14" />
+  <xacro:property name="arm_right_shoulder_roll_upper" value="3.14" />
+  <xacro:property name="arm_right_shoulder_roll_damping" value="0.0" />
+  <xacro:property name="arm_right_shoulder_roll_friction" value="0.0" />
+  <xacro:property name="arm_left_elbow_pitch_effort" value="18.0" />
+  <xacro:property name="arm_left_elbow_pitch_velocity" value="0.0" />
+  <xacro:property name="arm_left_elbow_pitch_lower" value="-3.14" />
+  <xacro:property name="arm_left_elbow_pitch_upper" value="3.14" />
+  <xacro:property name="arm_left_elbow_pitch_damping" value="0.0" />
+  <xacro:property name="arm_left_elbow_pitch_friction" value="0.0" />
+  <xacro:property name="arm_right_shoulder_pitch_effort" value="18.0" />
+  <xacro:property name="arm_right_shoulder_pitch_velocity" value="20.0" />
+  <xacro:property name="arm_right_shoulder_pitch_lower" value="-3.14" />
+  <xacro:property name="arm_right_shoulder_pitch_upper" value="3.14" />
+  <xacro:property name="arm_right_shoulder_pitch_damping" value="0.0" />
+  <xacro:property name="arm_right_shoulder_pitch_friction" value="0.0" />
+  <xacro:property name="knee_joint_right_effort" value="0.0" />
   <xacro:property name="knee_joint_right_velocity" value="12.0" />
   <xacro:property name="knee_joint_right_lower" value="-1.4" />
@@ -7,5 +43,23 @@
   <xacro:property name="knee_joint_right_damping" value="0.0" />
   <xacro:property name="knee_joint_right_friction" value="0.0" />
-  <xacro:property name="hip_pitch_right_effort" value="120.0" />
+  <xacro:property name="leg_right_hip_roll_effort" value="60.0" />
+  <xacro:property name="leg_right_hip_roll_velocity" value="10.0" />
+  <xacro:property name="leg_right_hip_roll_lower" value="-3.14" />
+  <xacro:property name="leg_right_hip_roll_upper" value="3.14" />
+  <xacro:property name="leg_right_hip_roll_damping" value="0.0" />
+  <xacro:property name="leg_right_hip_roll_friction" value="0.0" />
+  <xacro:property name="leg_left_hip_roll_effort" value="60.0" />
+  <xacro:property name="leg_left_hip_roll_velocity" value="0.0" />
+  <xacro:property name="leg_left_hip_roll_lower" value="-3.14" />
+  <xacro:property name="leg_left_hip_roll_upper" value="3.14" />
+  <xacro:property name="leg_left_hip_roll_damping" value="0.0" />
+  <xacro:property name="leg_left_hip_roll_friction" value="0.0" />
+  <xacro:property name="leg_right_knee_pitch_effort" value="120.0" />
+  <xacro:property name="leg_right_knee_pitch_velocity" value="12.0" />
+  <xacro:property name="leg_right_knee_pitch_lower" value="-3.14" />
+  <xacro:property name="leg_right_knee_pitch_upper" value="3.14" />
+  <xacro:property name="leg_right_knee_pitch_damping" value="0.0" />
+  <xacro:property name="leg_right_knee_pitch_friction" value="0.0" />
+  <xacro:property name="hip_pitch_right_effort" value="0.0" />
   <xacro:property name="hip_pitch_right_velocity" value="3.3" />
   <xacro:property name="hip_pitch_right_lower" value="-1.2" />
@@ -13,9 +67,51 @@
   <xacro:property name="hip_pitch_right_damping" value="0.0" />
   <xacro:property name="hip_pitch_right_friction" value="0.0" />
-  <xacro:property name="ankle_pitch_right_effort" value="18.0" />
-  <xacro:property name="ankle_pitch_right_velocity" value="10.0" />
+  <xacro:property name="leg_right_ankle_pitch_effort" value="30.0" />
+  <xacro:property name="leg_right_ankle_pitch_velocity" value="15.0" />
+  <xacro:property name="leg_right_ankle_pitch_lower" value="-3.14" />
+  <xacro:property name="leg_right_ankle_pitch_upper" value="3.14" />
+  <xacro:property name="leg_right_ankle_pitch_damping" value="0.0" />
+  <xacro:property name="leg_right_ankle_pitch_friction" value="0.0" />
+  <xacro:property name="leg_left_knee_pitch_effort" value="120.0" />
+  <xacro:property name="leg_left_knee_pitch_velocity" value="0.0" />
+  <xacro:property name="leg_left_knee_pitch_lower" value="-3.14" />
+  <xacro:property name="leg_left_knee_pitch_upper" value="3.14" />
+  <xacro:property name="leg_left_knee_pitch_damping" value="0.0" />
+  <xacro:property name="leg_left_knee_pitch_friction" value="0.0" />
+  <xacro:property name="leg_left_hip_pitch_effort" value="80.0" />
+  <xacro:property name="leg_left_hip_pitch_velocity" value="0.0" />
+  <xacro:property name="leg_left_hip_pitch_lower" value="-3.14" />
+  <xacro:property name="leg_left_hip_pitch_upper" value="3.14" />
+  <xacro:property name="leg_left_hip_pitch_damping" value="0.0" />
+  <xacro:property name="leg_left_hip_pitch_friction" value="0.0" />
+  <xacro:property name="ankle_pitch_right_effort" value="0.0" />
+  <xacro:property name="ankle_pitch_right_velocity" value="8.0" />
   <xacro:property name="ankle_pitch_right_lower" value="-0.8" />
   <xacro:property name="ankle_pitch_right_upper" value="0.8" />
   <xacro:property name="ankle_pitch_right_damping" value="0.0" />
   <xacro:property name="ankle_pitch_right_friction" value="0.0" />
+  <xacro:property name="arm_left_shoulder_pitch_effort" value="18.0" />
+  <xacro:property name="arm_left_shoulder_pitch_velocity" value="0.0" />
+  <xacro:property name="arm_left_shoulder_pitch_lower" value="-3.14" />
+  <xacro:property name="arm_left_shoulder_pitch_upper" value="3.14" />
+  <xacro:property name="arm_left_shoulder_pitch_damping" value="0.0" />
+  <xacro:property name="arm_left_shoulder_pitch_friction" value="0.0" />
+  <xacro:property name="leg_right_hip_yaw_effort" value="40.0" />
+  <xacro:property name="leg_right_hip_yaw_velocity" value="12.0" />
+  <xacro:property name="leg_right_hip_yaw_lower" value="-3.14" />
+  <xacro:property name="leg_right_hip_yaw_upper" value="3.14" />
+  <xacro:property name="leg_right_hip_yaw_damping" value="0.0" />
+  <xacro:property name="leg_right_hip_yaw_friction" value="0.0" />
+  <xacro:property name="arm_left_shoulder_roll_effort" value="18.0" />
+  <xacro:property name="arm_left_shoulder_roll_velocity" value="0.0" />
+  <xacro:property name="arm_left_shoulder_roll_lower" value="-3.14" />
+  <xacro:property name="arm_left_shoulder_roll_upper" value="3.14" />
+  <xacro:property name="arm_left_shoulder_roll_damping" value="0.0" />
+  <xacro:property name="arm_left_shoulder_roll_friction" value="0.0" />
+  <xacro:property name="arm_right_elbow_pitch_effort" value="18.0" />
+  <xacro:property name="arm_right_elbow_pitch_velocity" value="0.0" />
+  <xacro:property name="arm_right_elbow_pitch_lower" value="-3.14" />
+  <xacro:property name="arm_right_elbow_pitch_upper" value="3.14" />
+  <xacro:property name="arm_right_elbow_pitch_damping" value="0.0" />
+  <xacro:property name="arm_right_elbow_pitch_friction" value="0.0" />
 </robot>
